File: PCB (KiCAD)/Cooee_keyboard.kicad_sch (KiCad schematic)
At the start: 105 parts, among them J1 Conn_01x15_Pin, Sw555 {dblquote}

Commit message: changed computer PCB edge shape to match keyboard
So these can be 2x 2layer boards back to back, easy PnP/hotplate assembly, more modular (replaceable keyboards)
Parts:
- J1: now left out of the parts list
Changed lines of the file:
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@@
 		(unit 1)
 		(exclude_from_sim no)
-		(in_bom yes)
+		(in_bom no)
 		(on_board yes)
 		(dnp no)
