File: PCB (KiCAD)/Cooee_brains.kicad_pcb (KiCad board)
At the start: 2 copper layers, 66.8 x 65.3 mm, 73 parts, among them J1 USB4105-GF-A, J2 Conn_Coaxial, J3 503398-1892, J4 Conn_01x14_Socket, J5 Conn_01x02_Pin, J6 Conn_Coaxial, J7 Conn_01x04_Pin, J9 Conn_01x05_Socket, SW1 Prog, SW2 Reset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

Commit message: fixed up some incorrect footprints/symbols
fixed up some incorrect footprints/symbols
Parts:
- removed MK1: INMP441, USB4105-GF-A (1):MIC_INMP441
- removed R12: 10kΩ, Capacitor_SMD:C_0805_2012Metric_Pad1.18x1.45mm_HandSolder
- removed RProg1: 330, Capacitor_SMD:C_0805_2012Metric_Pad1.18x1.45mm_HandSolder
- added C12: 100nF, Capacitor_SMD:C_0805_2012Metric, B.Cu at (149.7, 99.2)
- added D2: D, Diode_SMD:D_0805_2012Metric_Pad1.15x1.40mm_HandSolder, B.Cu at (163.9, 84.0)
- added J10: Conn_01x02_Pin, Connector_PinHeader_2.54mm:PinHeader_1x02_P2.54mm_Horizontal, F.Cu at (187.4, 69.6)
- added J11: Conn_01x02_Pin, Connector_PinHeader_2.54mm:PinHeader_1x02_P2.54mm_Horizontal, F.Cu at (129.9, 115.9)
- added J8: Conn_01x02_Pin, Connector_PinHeader_2.54mm:PinHeader_1x02_P2.54mm_Horizontal, B.Cu at (162.2, 81.8)
- added MK2: ICS-43434, USB4105-GF-A (1):MIC_ICS-43434, B.Cu at (153.5, 102.2)
- added R21: 2kΩ, Capacitor_SMD:C_0805_2012Metric_Pad1.18x1.45mm_HandSolder, B.Cu at (142.4, 121.1)
- added R22: 330, Capacitor_SMD:C_0805_2012Metric_Pad1.18x1.45mm_HandSolder, B.Cu at (164.6, 79.2)
- added R23: 10kΩ, Capacitor_SMD:C_0805_2012Metric_Pad1.18x1.45mm_HandSolder, B.Cu at (151.3, 104.9)
- TP1: value TestPoint -> Display CS
- TP11: value TestPoint -> 3.3V
- TP12: value TestPoint -> Keyboard Data
- TP13: value TestPoint -> Keyboard Clock
- TP4: value TestPoint -> MOSI
- TP5: value TestPoint -> MISO
- TP6: value TestPoint -> CLCK
- U3: footprint Package_DFN_QFN:QFN-24-1EP_4x4mm_P0.5mm_EP2.6x2.6mm -> Package_DFN_QFN:TQFN-16-1EP_3x3mm_P0.5mm_EP1.6x1.6mm
- moved R16 0.32 mm to (166.8, 83.0), turned to 90 degrees
Connections:
- net SPARE1 renamed TALK_SW
- U2 pad 20: LoRa_DIO1 -> LoRa_DIO0
- U2 pad 25: MIC_EN -> LoRa_DIO1
- U2 pad 39: unconnected-(U2-IO1-Pad39) -> LoRa_DIO2
- U3 pad 17: SPKR_EN -> GND
- U7 pad 9: unconnected-(U7-EP-Pad9) -> GND
- U8 pad 5: LoRa_DIO1 -> LoRa_DIO0
- U8 pad 6: LoRa_DIO2 -> LoRa_DIO1
- U8 pad 7: unconnected-(U8-DIO2-Pad7) -> LoRa_DIO2
Routing:
- net LoRa_DIO2: track 0.00 -> 68.9 mm, vias 0 -> 4
- net LoRa_DIO0: track 0.00 -> 57.4 mm, vias 0 -> 2
- net TALK_SW: track 8.88 -> 53.3 mm, vias 1 -> 2
- net Net-(J10-Pin_1): track 13.1 -> 42.8 mm
- net GND: track 103.3 -> 127.2 mm, vias 72 -> 78
- net MIC_EN: track 20.6 -> 0.00 mm
- net LoRa_DIO1: track 57.5 -> 37.5 mm
- net Net-(J11-Pin_1): track 0.00 -> 14.0 mm
- net (no net): track 13.7 -> 7.49 mm
- net SPEAKER+: track 17.9 -> 22.9 mm, vias 0 -> 1
- net SPKR_LRCK: track 24.0 -> 19.7 mm
- net SPEAKER-: track 17.1 -> 20.8 mm, vias 0 -> 1
- net KEEB_INT: track 43.6 -> 40.3 mm
- net KEEB_SCL: track 61.9 -> 59.0 mm
- net 5V: track 85.0 -> 87.8 mm
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Other:
- outline, holes or cut-outs redrawn
- board text added: "+"
- board text added: "-"
- board text added: "-- ++"
- board text added: "3.3V"
- board text added: "< --- Disable Thermal"
- board text added: "BATT NEGATIVE"
- board text added: "COOEE"
- board text added: "GPS Module"
- board text added: "KEYBOARD"
- board text added: "MIC->"
- board text added: "Speaker"
- board text added: "Talk SW"
- board text added: "Thermister"
- board text added: "USB Interface Bypass"
- board text added: "Visit: Github.com/DetectiveMittens/Cooee/"
- board text removed: "SCK"
- board text removed: "SPACE FOR BATTERY"
- board text removed: "SPACE FOR SPEAKER"
